File: KiCad/Nixie/Nixie.sch (KiCad schematic (older format))
At the start: 33 parts

Commit message: First PCB draft
Parts:
- removed J?: Conn_01x03_Female, symbol Connector:Conn_01x03_Female
- removed J?: Conn_01x03_Male, symbol Connector:Conn_01x03_Male
- removed J?: Conn_01x05_Female, symbol Connector:Conn_01x05_Female
- removed J?: Conn_01x05_Male, symbol Connector:Conn_01x05_Male
- added J2: DB9_Male_MountingHoles, Connector_Dsub:DSUB-9_Female_Horizontal_P2.77x2.84mm_EdgePinOffset7.70mm_Housed_MountingHolesOffset9.12mm, symbol Connector:DB9_Male_MountingHoles
- added J3: DB9_Female_MountingHoles, Connector_Dsub:DSUB-9_Male_Horizontal_P2.77x2.84mm_EdgePinOffset7.70mm_Housed_MountingHolesOffset9.12mm, symbol Connector:DB9_Female_MountingHoles
- C1, C3: renamed from C?; footprint (none) -> Capacitor_SMD:C_0805_2012Metric
- C2: renamed from C?; footprint (none) -> Capacitor_SMD:CP_Elec_10x12.5
- C4: renamed from C?; footprint (none) -> Capacitor_SMD:CP_Elec_4x5.4
- J1: renamed from J?; footprint (none) -> Connector_Phoenix_MC_HighVoltage:PhoenixContact_MCV_1,5_2-G-5.08_1x02_P5.08mm_Vertical
- NIX1: renamed from NIX?; footprint (none) -> Valve:Z5730M
- Q1, Q10, Q2, Q3, Q4, Q5, Q6, Q7, Q8, Q9: renamed from Q?; footprint Package_TO_SOT_THT:TO-92_Inline -> Package_TO_SOT_SMD:SOT-23
- R1, R10, R11, R2, R3, R4, R5, R7, R8, R9: renamed from R?; footprint (none) -> Resistor_SMD:R_0805_2012Metric
- R6: renamed from R?; footprint (none) -> Resistor_THT:R_Axial_DIN0617_L17.0mm_D6.0mm_P7.62mm_Vertical
- U1: renamed from U?; footprint (none) -> Package_SO:SOP-16_4.55x10.3mm_P1.27mm
- U2: renamed from U?; footprint (none) -> Package_SO:SOIC-16_3.9x9.9mm_P1.27mm
Connections:
- net +170V: now also J2.5, J3.1
- net +5V: now also J2.3, J3.3
- net CLK: now also J2.2, J3.4
- net DATA_IN: now also J2.6
- net DATA_OUT: now also J3.9
- net GND: now also J2.0 (PAD), J2.1, J3.0 (PAD), J3.5
- net LATCH: now also J2.7, J3.8
- no-connect marks 6 -> 10
Other:
- moved on the sheet: C1, C2, C3, C4, J1

Commit message: PCB routing part 1
Connections:
- net +170V: now also J3.5; no longer J3.1
- net CLK: now also J3.2; no longer J3.4
- net DATA_OUT: now also J3.6; no longer J3.9
- net GND: now also J3.1; no longer J3.5
- net LATCH: now also J3.7; no longer J3.8
Other:
- moved on the sheet: J3
Changed lines of the file:
@@
 L power:+5V #PWR?
 U 1 1 5D560501
-P 2500 2300
-F 0 "#PWR?" H 2500 2150 50  0001 C CNN
-F 1 "+5V" H 2515 2473 50  0000 C CNN
-F 2 "" H 2500 2300 50  0001 C CNN
-F 3 "" H 2500 2300 50  0001 C CNN
-	1    2500 2300
+P 2600 2300
+F 0 "#PWR?" H 2600 2150 50  0001 C CNN
+F 1 "+5V" H 2615 2473 50  0000 C CNN
+F 2 "" H 2600 2300 50  0001 C CNN
+F 3 "" H 2600 2300 50  0001 C CNN
+	1    2600 2300
 	1    0    0    -1
 $EndComp
@@
 L power:GND #PWR?
 U 1 1 5D560BCA
-P 2500 2900
-F 0 "#PWR?" H 2500 2650 50  0001 C CNN
-F 1 "GND" H 2505 2727 50  0000 C CNN
-F 2 "" H 2500 2900 50  0001 C CNN
-F 3 "" H 2500 2900 50  0001 C CNN
-	1    2500 2900
-	1    0    0    -1
-$EndComp
-Wire Wire Line
-	2500 2800 2500 2900
-Wire Wire Line
-	2500 2400 2500 2300
+P 2600 2900
+F 0 "#PWR?" H 2600 2650 50  0001 C CNN
+F 1 "GND" H 2605 2727 50  0000 C CNN
+F 2 "" H 2600 2900 50  0001 C CNN
+F 3 "" H 2600 2900 50  0001 C CNN
+	1    2600 2900
+	1    0    0    -1
+$EndComp
+Wire Wire Line
+	2600 2000 2600 1900
 Wire Wire Line
 	2950 5200 3350 5200
@@
 Text Label 1650 2700 0    50   ~ 0
 DATA_IN
-Text Label 2500 2700 2    50   ~ 0
+Text Label 2600 2700 2    50   ~ 0
 DATA_OUT
-Text Label 2500 2600 2    50   ~ 0
+Text Label 2600 2600 2    50   ~ 0
 CLK
-Text Label 2500 2500 2    50   ~ 0
+Text Label 2600 2500 2    50   ~ 0
 LATCH
 $Comp
@@
 L Nixie-rescue:+170V-power #PWR?
 U 1 1 5D60968C
-P 2500 1900
-F 0 "#PWR?" H 2500 1750 50  0001 C CNN
-F 1 "+170V" H 2515 2073 50  0000 C CNN
-F 2 "" H 2500 1900 50  0001 C CNN
-F 3 "" H 2500 1900 50  0001 C CNN
-	1    2500 1900
-	1    0    0    -1
-$EndComp
-Wire Wire Line
-	2500 1900 2500 2000
+P 2600 1900
+F 0 "#PWR?" H 2600 1750 50  0001 C CNN
+F 1 "+170V" H 2615 2073 50  0000 C CNN
+F 2 "" H 2600 1900 50  0001 C CNN
+F 3 "" H 2600 1900 50  0001 C CNN
+	1    2600 1900
+	1    0    0    -1
+$EndComp
+Wire Wire Line
+	2600 2900 2600 2800
 $Comp
 L Nixie-rescue:+170V-power #PWR?
@@
 Connection ~ 1650 2800
 $Comp
-L Connector:DB9_Female_MountingHoles J3
-U 1 1 5D3FDF15
-P 3050 2400
-F 0 "J3" H 3230 2356 50  0000 L CNN
-F 1 "DB9_Female_MountingHoles" H 3230 2311 50  0001 L CNN
-F 2 "Connector_Dsub:DSUB-9_Male_Horizontal_P2.77x2.84mm_EdgePinOffset7.70mm_Housed_MountingHolesOffset9.12mm" H 3050 2400 50  0001 C CNN
-F 3 " ~" H 3050 2400 50  0001 C CNN
-	1    3050 2400
-	1    0    0    -1
-$EndComp
-$Comp
 L Connector:DB9_Male_MountingHoles J2
 U 1 1 5D406C9F
@@
 L power:GND #PWR?
 U 1 1 5D4476A3
-P 3050 3100
-F 0 "#PWR?" H 3050 2850 50  0001 C CNN
-F 1 "GND" H 3055 2927 50  0000 C CNN
-F 2 "" H 3050 3100 50  0001 C CNN
-F 3 "" H 3050 3100 50  0001 C CNN
-	1    3050 3100
-	1    0    0    -1
-$EndComp
-Wire Wire Line
-	3050 3100 3050 3000
+P 3150 1700
+F 0 "#PWR?" H 3150 1450 50  0001 C CNN
+F 1 "GND" H 3155 1527 50  0000 C CNN
+F 2 "" H 3150 1700 50  0001 C CNN
+F 3 "" H 3150 1700 50  0001 C CNN
+	1    3150 1700
+	1    0    0    1
+$EndComp
+Wire Wire Line
+	3150 1700 3150 1800
 Wire Wire Line
 	1400 2800 1650 2800
 Wire Wire Line
-	2500 2800 2750 2800
-Wire Wire Line
-	2500 2700 2750 2700
-Wire Wire Line
-	2500 2600 2750 2600
-Wire Wire Line
-	2500 2500 2750 2500
-Wire Wire Line
-	2500 2400 2750 2400
+	2600 2000 2850 2000
 Wire Wire Line
 	1400 2700 1650 2700
@@
 	1400 2000 1650 2000
 Wire Wire Line
-	2500 2000 2750 2000
+	2600 2800 2850 2800
 NoConn ~ 1400 2100
 NoConn ~ 1400 2200
 NoConn ~ 1400 2300
-NoConn ~ 2750 2100
-NoConn ~ 2750 2200
-NoConn ~ 2750 2300
+$Comp
+L Connector:DB9_Female_MountingHoles J3
+U 1 1 5D3FDF15
+P 3150 2400
+F 0 "J3" H 3330 2356 50  0000 L CNN
+F 1 "DB9_Female_MountingHoles" H 3330 2311 50  0001 L CNN
+F 2 "Connector_Dsub:DSUB-9_Male_Horizontal_P2.77x2.84mm_EdgePinOffset7.70mm_Housed_MountingHolesOffset9.12mm" H 3150 2400 50  0001 C CNN
+F 3 " ~" H 3150 2400 50  0001 C CNN
+	1    3150 2400
+	1    0    0    1
+$EndComp
+Wire Wire Line
+	2600 2300 2600 2400
+Wire Wire Line
+	2600 2400 2850 2400
+Wire Wire Line
+	2850 2500 2600 2500
+Wire Wire Line
+	2600 2600 2850 2600
+Wire Wire Line
+	2850 2700 2600 2700
+NoConn ~ 2850 2100
+NoConn ~ 2850 2200
+NoConn ~ 2850 2300
 $EndSCHEMATC

Commit message: Finished the board
Parts:
- R1, R10, R11, R2, R3, R4, R5, R7, R8, R9: value 50k -> 47k
Changed lines of the file:
@@
 EESchema Schematic File Version 4
 LIBS:Nixie-cache
-EELAYER 29 0
+EELAYER 30 0
 EELAYER END
 $Descr A4 11693 8268
@@
 P 4550 4700
 F 0 "R1" H 4620 4746 50  0000 L CNN
-F 1 "50k" H 4620 4655 50  0000 L CNN
+F 1 "47k" H 4620 4655 50  0000 L CNN
 F 2 "Resistor_SMD:R_0805_2012Metric" V 4480 4700 50  0001 C CNN
 F 3 "~" H 4550 4700 50  0001 C CNN
@@
 P 5250 4700
 F 0 "R2" H 5320 4746 50  0000 L CNN
-F 1 "50k" H 5320 4655 50  0000 L CNN
+F 1 "47k" H 5320 4655 50  0000 L CNN
 F 2 "Resistor_SMD:R_0805_2012Metric" V 5180 4700 50  0001 C CNN
 F 3 "~" H 5250 4700 50  0001 C CNN
@@
 P 5850 4700
 F 0 "R3" H 5920 4746 50  0000 L CNN
-F 1 "50k" H 5920 4655 50  0000 L CNN
+F 1 "47k" H 5920 4655 50  0000 L CNN
 F 2 "Resistor_SMD:R_0805_2012Metric" V 5780 4700 50  0001 C CNN
 F 3 "~" H 5850 4700 50  0001 C CNN
@@
 P 6450 4700
 F 0 "R4" H 6520 4746 50  0000 L CNN
-F 1 "50k" H 6520 4655 50  0000 L CNN
+F 1 "47k" H 6520 4655 50  0000 L CNN
 F 2 "Resistor_SMD:R_0805_2012Metric" V 6380 4700 50  0001 C CNN
 F 3 "~" H 6450 4700 50  0001 C CNN
@@
 P 7050 4700
 F 0 "R5" H 7120 4746 50  0000 L CNN
-F 1 "50k" H 7120 4655 50  0000 L CNN
+F 1 "47k" H 7120 4655 50  0000 L CNN
 F 2 "Resistor_SMD:R_0805_2012Metric" V 6980 4700 50  0001 C CNN
 F 3 "~" H 7050 4700 50  0001 C CNN
@@
 P 7650 4700
 F 0 "R7" H 7720 4746 50  0000 L CNN
-F 1 "50k" H 7720 4655 50  0000 L CNN
+F 1 "47k" H 7720 4655 50  0000 L CNN
 F 2 "Resistor_SMD:R_0805_2012Metric" V 7580 4700 50  0001 C CNN
 F 3 "~" H 7650 4700 50  0001 C CNN
@@
 P 8250 4700
 F 0 "R8" H 8320 4746 50  0000 L CNN
-F 1 "50k" H 8320 4655 50  0000 L CNN
+F 1 "47k" H 8320 4655 50  0000 L CNN
 F 2 "Resistor_SMD:R_0805_2012Metric" V 8180 4700 50  0001 C CNN
 F 3 "~" H 8250 4700 50  0001 C CNN
@@
 P 8850 4700
 F 0 "R9" H 8920 4746 50  0000 L CNN
-F 1 "50k" H 8920 4655 50  0000 L CNN
+F 1 "47k" H 8920 4655 50  0000 L CNN
 F 2 "Resistor_SMD:R_0805_2012Metric" V 8780 4700 50  0001 C CNN
 F 3 "~" H 8850 4700 50  0001 C CNN
@@
 P 9450 4700
 F 0 "R10" H 9520 4746 50  0000 L CNN
-F 1 "50k" H 9520 4655 50  0000 L CNN
+F 1 "47k" H 9520 4655 50  0000 L CNN
 F 2 "Resistor_SMD:R_0805_2012Metric" V 9380 4700 50  0001 C CNN
 F 3 "~" H 9450 4700 50  0001 C CNN
@@
 P 10050 4700
 F 0 "R11" H 10120 4746 50  0000 L CNN
-F 1 "50k" H 10120 4655 50  0000 L CNN
+F 1 "47k" H 10120 4655 50  0000 L CNN
 F 2 "Resistor_SMD:R_0805_2012Metric" V 9980 4700 50  0001 C CNN
 F 3 "~" H 10050 4700 50  0001 C CNN
