File: KiCad/Nixie/Nixie.sch (KiCad schematic (older format))
At the start: 31 parts, among them J0 DB9_Male_MountingHoles, J1 Screw_Terminal_01x02, J2 DB9_Female_MountingHoles, Q0 Q_NPN_BEC, Q1 Q_NPN_BEC, Q2 Q_NPN_BEC, Q3 Q_NPN_BEC, Q4 Q_NPN_BEC, Q5 Q_NPN_BEC, Q6 Q_NPN_BEC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

Commit message: Minor Schematic Change
Parts:
- NIX0: symbol nixie:NixieTube -> Nixie-rescue:NixieTube-nixie
Other:
- moved on the sheet: C0, C1, C2, C3, U0
Changed lines of the file:
@@
 EESchema Schematic File Version 4
-LIBS:Nixie-cache
 EELAYER 30 0
 EELAYER END
@@
 $EndDescr
 $Comp
-L nixie:NixieTube NIX0
+L Nixie-rescue:NixieTube-nixie NIX0
 U 1 1 5D3DF708
 P 7350 3450
@@
 L 74xx:74HC595 U0
 U 1 1 5D3E3D4A
-P 2200 5400
-F 0 "U0" H 2200 6181 50  0000 C CNN
-F 1 "74HC595" H 2200 6090 50  0000 C CNN
-F 2 "Package_SO:SOP-16_4.55x10.3mm_P1.27mm" H 2200 5400 50  0001 C CNN
-F 3 "http://www.ti.com/lit/ds/symlink/sn74hc595.pdf" H 2200 5400 50  0001 C CNN
-	1    2200 5400
+P 2100 5600
+F 0 "U0" H 2100 6381 50  0000 C CNN
+F 1 "74HC595" H 2100 6290 50  0000 C CNN
+F 2 "Package_SO:SOP-16_4.55x10.3mm_P1.27mm" H 2100 5600 50  0001 C CNN
+F 3 "http://www.ti.com/lit/ds/symlink/sn74hc595.pdf" H 2100 5600 50  0001 C CNN
+	1    2100 5600
 	1    0    0    -1
 $EndComp
@@
 L Device:C C2
 U 1 1 5D3F6AE2
-P 3950 2450
-F 0 "C2" H 4065 2496 50  0000 L CNN
-F 1 "100n" H 4065 2405 50  0000 L CNN
-F 2 "Capacitor_SMD:C_0805_2012Metric" H 3988 2300 50  0001 C CNN
-F 3 "~" H 3950 2450 50  0001 C CNN
-	1    3950 2450
+P 4600 2450
+F 0 "C2" H 4715 2496 50  0000 L CNN
+F 1 "100n" H 4715 2405 50  0000 L CNN
+F 2 "Capacitor_SMD:C_0805_2012Metric" H 4638 2300 50  0001 C CNN
+F 3 "~" H 4600 2450 50  0001 C CNN
+	1    4600 2450
 	1    0    0    -1
 $EndComp
@@
 L Device:C C0
 U 1 1 5D3F7976
-P 3550 2450
-F 0 "C0" H 3665 2496 50  0000 L CNN
-F 1 "100n" H 3665 2405 50  0000 L CNN
-F 2 "Capacitor_SMD:C_0805_2012Metric" H 3588 2300 50  0001 C CNN
-F 3 "~" H 3550 2450 50  0001 C CNN
-	1    3550 2450
+P 4200 2450
+F 0 "C0" H 4315 2496 50  0000 L CNN
+F 1 "100n" H 4315 2405 50  0000 L CNN
+F 2 "Capacitor_SMD:C_0805_2012Metric" H 4238 2300 50  0001 C CNN
+F 3 "~" H 4200 2450 50  0001 C CNN
+	1    4200 2450
 	1    0    0    -1
 $EndComp
@@
 L power:GND #PWR?
 U 1 1 5D4BF5BF
-P 2200 6200
-F 0 "#PWR?" H 2200 5950 50  0001 C CNN
-F 1 "GND" H 2205 6027 50  0000 C CNN
-F 2 "" H 2200 6200 50  0001 C CNN
-F 3 "" H 2200 6200 50  0001 C CNN
-	1    2200 6200
+P 2100 6400
+F 0 "#PWR?" H 2100 6150 50  0001 C CNN
+F 1 "GND" H 2105 6227 50  0000 C CNN
+F 2 "" H 2100 6400 50  0001 C CNN
+F 3 "" H 2100 6400 50  0001 C CNN
+	1    2100 6400
 	1    0    0    -1
 $EndComp
@@
 L power:+5V #PWR?
 U 1 1 5D4C45D8
-P 2200 4700
-F 0 "#PWR?" H 2200 4550 50  0001 C CNN
-F 1 "+5V" H 2215 4873 50  0000 C CNN
-F 2 "" H 2200 4700 50  0001 C CNN
-F 3 "" H 2200 4700 50  0001 C CNN
-	1    2200 4700
+P 2100 4900
+F 0 "#PWR?" H 2100 4750 50  0001 C CNN
+F 1 "+5V" H 2115 5073 50  0000 C CNN
+F 2 "" H 2100 4900 50  0001 C CNN
+F 3 "" H 2100 4900 50  0001 C CNN
+	1    2100 4900
 	1    0    0    -1
 $EndComp
@@
 	3850 4600 3850 4700
 Wire Wire Line
-	2200 4700 2200 4800
-Wire Wire Line
-	2200 6100 2200 6200
+	2100 4900 2100 5000
+Wire Wire Line
+	2100 6300 2100 6400
 $Comp
 L power:GND #PWR?
@@
 Wire Wire Line
 	2600 2000 2600 1900
-Wire Wire Line
-	2950 5200 3350 5200
-Wire Wire Line
-	2950 5200 2950 5000
-Wire Wire Line
-	2950 5000 2600 5000
-Wire Wire Line
-	2600 5100 2850 5100
-Wire Wire Line
-	2850 5100 2850 5300
-Wire Wire Line
-	2850 5300 3350 5300
-Wire Wire Line
-	2750 5400 2750 5200
-Wire Wire Line
-	2750 5200 2600 5200
-Wire Wire Line
-	2750 5400 3350 5400
-Wire Wire Line
-	2600 5300 2700 5300
-Wire Wire Line
-	2700 5300 2700 5500
-Wire Wire Line
-	2700 5500 3350 5500
-NoConn ~ 2600 5400
-NoConn ~ 2600 5500
-NoConn ~ 2600 5600
-NoConn ~ 2600 5700
+NoConn ~ 2500 5600
+NoConn ~ 2500 5700
+NoConn ~ 2500 5800
+NoConn ~ 2500 5900
 Text Label 1650 2500 0    50   ~ 0
 LATCH
@@
 L Device:CP C3
 U 1 1 5D62A740
-P 4350 2450
-F 0 "C3" H 4468 2496 50  0000 L CNN
-F 1 "10u" H 4468 2405 50  0000 L CNN
-F 2 "Capacitor_SMD:CP_Elec_4x5.4" H 4388 2300 50  0001 C CNN
-F 3 "~" H 4350 2450 50  0001 C CNN
-	1    4350 2450
-	1    0    0    -1
-$EndComp
-Connection ~ 3950 2300
-Connection ~ 3950 2600
+P 5000 2450
+F 0 "C3" H 5118 2496 50  0000 L CNN
+F 1 "10u" H 5118 2405 50  0000 L CNN
+F 2 "Capacitor_SMD:CP_Elec_4x5.4" H 5038 2300 50  0001 C CNN
+F 3 "~" H 5000 2450 50  0001 C CNN
+	1    5000 2450
+	1    0    0    -1
+$EndComp
+Connection ~ 4600 2300
+Connection ~ 4600 2600
 $Comp
 L power:GND #PWR?
 U 1 1 5D63569F
-P 3950 2700
-F 0 "#PWR?" H 3950 2450 50  0001 C CNN
-F 1 "GND" H 3955 2527 50  0000 C CNN
-F 2 "" H 3950 2700 50  0001 C CNN
-F 3 "" H 3950 2700 50  0001 C CNN
-	1    3950 2700
+P 4600 2700
+F 0 "#PWR?" H 4600 2450 50  0001 C CNN
+F 1 "GND" H 4605 2527 50  0000 C CNN
+F 2 "" H 4600 2700 50  0001 C CNN
+F 3 "" H 4600 2700 50  0001 C CNN
+	1    4600 2700
 	1    0    0    -1
 $EndComp
@@
 L power:+5V #PWR?
 U 1 1 5D635F4B
-P 3950 2200
-F 0 "#PWR?" H 3950 2050 50  0001 C CNN
-F 1 "+5V" H 3965 2373 50  0000 C CNN
-F 2 "" H 3950 2200 50  0001 C CNN
-F 3 "" H 3950 2200 50  0001 C CNN
-	1    3950 2200
-	1    0    0    -1
-$EndComp
-Wire Wire Line
-	3950 2200 3950 2300
-Wire Wire Line
-	3950 2600 3950 2700
+P 4600 2200
+F 0 "#PWR?" H 4600 2050 50  0001 C CNN
+F 1 "+5V" H 4615 2373 50  0000 C CNN
+F 2 "" H 4600 2200 50  0001 C CNN
+F 3 "" H 4600 2200 50  0001 C CNN
+	1    4600 2200
+	1    0    0    -1
+$EndComp
+Wire Wire Line
+	4600 2200 4600 2300
+Wire Wire Line
+	4600 2600 4600 2700
 $Comp
 L Device:CP C1
 U 1 1 5D640535
-P 3950 1450
-F 0 "C1" H 4068 1496 50  0000 L CNN
-F 1 "10u" H 4068 1405 50  0000 L CNN
-F 2 "Capacitor_SMD:CP_Elec_10x12.5" H 3988 1300 50  0001 C CNN
-F 3 "~" H 3950 1450 50  0001 C CNN
-	1    3950 1450
+P 4600 1450
+F 0 "C1" H 4718 1496 50  0000 L CNN
+F 1 "10u" H 4718 1405 50  0000 L CNN
+F 2 "Capacitor_SMD:CP_Elec_10x12.5" H 4638 1300 50  0001 C CNN
+F 3 "~" H 4600 1450 50  0001 C CNN
+	1    4600 1450
 	1    0    0    -1
 $EndComp
@@
 L power:GND #PWR?
 U 1 1 5D643206
-P 3950 1700
-F 0 "#PWR?" H 3950 1450 50  0001 C CNN
-F 1 "GND" H 3955 1527 50  0000 C CNN
-F 2 "" H 3950 1700 50  0001 C CNN
-F 3 "" H 3950 1700 50  0001 C CNN
-	1    3950 1700
+P 4600 1700
+F 0 "#PWR?" H 4600 1450 50  0001 C CNN
+F 1 "GND" H 4605 1527 50  0000 C CNN
+F 2 "" H 4600 1700 50  0001 C CNN
+F 3 "" H 4600 1700 50  0001 C CNN
+	1    4600 1700
 	1    0    0    -1
 $EndComp
@@
 L Nixie-rescue:+170V-power #PWR?
 U 1 1 5D64429C
-P 3950 1200
-F 0 "#PWR?" H 3950 1050 50  0001 C CNN
-F 1 "+170V" H 3965 1373 50  0000 C CNN
-F 2 "" H 3950 1200 50  0001 C CNN
-F 3 "" H 3950 1200 50  0001 C CNN
-	1    3950 1200
-	1    0    0    -1
-$EndComp
-Wire Wire Line
-	3950 1200 3950 1300
-Wire Wire Line
-	3950 1600 3950 1700
+P 4600 1200
+F 0 "#PWR?" H 4600 1050 50  0001 C CNN
+F 1 "+170V" H 4615 1373 50  0000 C CNN
+F 2 "" H 4600 1200 50  0001 C CNN
+F 3 "" H 4600 1200 50  0001 C CNN
+	1    4600 1200
+	1    0    0    -1
+$EndComp
+Wire Wire Line
+	4600 1200 4600 1300
+Wire Wire Line
+	4600 1600 4600 1700
 $Comp
 L Nixie-rescue:+170V-power #PWR?
@@
 Wire Wire Line
 	7650 2150 7650 2300
-Text Label 2700 5900 0    50   ~ 0
+Text Label 2600 6100 0    50   ~ 0
 DATA_OUT
 Wire Wire Line
-	2700 5900 2600 5900
-Wire Wire Line
-	1800 5600 1700 5600
-Wire Wire Line
-	1700 5600 1700 6100
-Wire Wire Line
-	1700 6100 2200 6100
-Connection ~ 2200 6100
-Text Label 1600 5500 2    50   ~ 0
-LATCH
-Connection ~ 2200 4800
-Text Label 1700 5200 2    50   ~ 0
+	2600 6100 2500 6100
+Wire Wire Line
+	1200 5800 1200 6300
+Connection ~ 2100 6300
+Connection ~ 2100 5000
+Text Label 1600 5400 2    50   ~ 0
 CLK
-Wire Wire Line
-	1600 5500 1800 5500
-Text Label 1700 5000 2    50   ~ 0
+Text Label 1600 5200 2    50   ~ 0
 DATA_IN
 Wire Wire Line
-	1700 5000 1800 5000
-Wire Wire Line
-	1800 5200 1700 5200
-Wire Wire Line
-	1300 5300 1300 4800
-Wire Wire Line
-	1300 5300 1800 5300
-Wire Wire Line
-	1300 4800 2200 4800
-Wire Wire Line
-	3550 2300 3950 2300
-Wire Wire Line
-	3950 2300 4350 2300
-Wire Wire Line
-	3950 2600 4350 2600
-Wire Wire Line
-	3550 2600 3950 2600
+	1600 5200 1700 5200
+Wire Wire Line
+	1700 5400 1600 5400
+Wire Wire Line
+	1200 5500 1200 5000
+Wire Wire Line
+	1200 5500 1700 5500
+Wire Wire Line
+	1200 5000 2100 5000
+Wire Wire Line
+	4200 2300 4600 2300
+Wire Wire Line
+	4600 2300 5000 2300
+Wire Wire Line
+	4600 2600 5000 2600
+Wire Wire Line
+	4200 2600 4600 2600
 $Comp
 L Device:R R0
@@
 	1    0    0    -1
 $EndComp
+Wire Wire Line
+	2500 5200 3350 5200
+Wire Wire Line
+	2500 5300 3350 5300
+Wire Wire Line
+	2500 5400 3350 5400
+Wire Wire Line
+	3350 5500 2500 5500
+Wire Wire Line
+	1200 5800 1700 5800
+Wire Wire Line
+	1200 6300 2100 6300
+Text Label 1600 5700 2    50   ~ 0
+LATCH
+Wire Wire Line
+	1600 5700 1700 5700
 $EndSCHEMATC
