File: KiCad/Nixie/Nixie.kicad_pcb (KiCad board)
At the start: 2 copper layers, 33 x 73.7 mm, 31 parts, among them J1 Screw_Terminal_01x02, J2 DB9_Male_MountingHoles, J3 DB9_Female_MountingHoles, Q1 MMBTA42, Q10 MMBTA42, Q2 MMBTA42, Q3 MMBTA42, Q4 MMBTA42, Q5 MMBTA42, Q6 MMBTA42, Q7 MMBTA42, Q8 MMBTA42, Q9 MMBTA42, U1 74HC595, U2 4028

Commit message: PCB routing part 1
Parts:
- NIX1: moved to B.Cu
- moved R8 30.5 mm to (130.0, 43.2)
- moved R2 30.1 mm to (153.2, 64.0), turned to 90 degrees
- moved R10 27.6 mm to (153.2, 68.8), turned to 90 degrees
- moved R4 23.3 mm to (153.2, 59.1), turned to 90 degrees
- moved Q1 22.6 mm to (129.0, 85.6), turned to 90 degrees
- moved R9 20.4 mm to (130.0, 50.0)
- moved R11 19.3 mm to (130.0, 47.8)
- moved C3 14.1 mm to (155.2, 58.2), turned to 270 degrees
- moved J3 12.3 mm to (142.2, 64.5), turned to 90 degrees
- moved J2 12.2 mm to (137.4, 64.5), turned to 270 degrees
- moved R7 4.83 mm to (130.0, 45.5)
- moved R1 4.83 mm to (130.0, 52.3)
- moved R5 3.06 mm to (130.0, 56.9)
- moved R3 2.30 mm to (130.0, 54.6)
Connections:
- J3 pad 1: +170V -> GND
- J3 pad 2: Net-(J3-Pad2) -> /CLK
- J3 pad 4: /CLK -> Net-(J3-Pad4)
- J3 pad 5: GND -> +170V
- J3 pad 6: Net-(J3-Pad6) -> /DATA_OUT
- J3 pad 7: Net-(J3-Pad7) -> /LATCH
- J3 pad 8: /LATCH -> Net-(J3-Pad8)
- J3 pad 9: /DATA_OUT -> Net-(J3-Pad9)
Routing:
- net +170V: track 0.00 -> 66.5 mm
- net /LATCH: track 0.00 -> 54.2 mm, vias 0 -> 6
- net /CLK: track 0.00 -> 50.1 mm, vias 0 -> 4
- net +5V: track 0.00 -> 46.2 mm
- net /DATA_IN: track 0.00 -> 41.9 mm, vias 0 -> 6
- net /DATA_OUT: track 0.00 -> 37.6 mm, vias 0 -> 2
- net Net-(R5-Pad2): track 0.00 -> 24.3 mm
- net Net-(R10-Pad2): track 0.00 -> 23.5 mm
- net Net-(R3-Pad2): track 0.00 -> 22.6 mm
- net Net-(R7-Pad2): track 0.00 -> 22.1 mm
- net Net-(R8-Pad2): track 0.00 -> 21.7 mm
- net Net-(R1-Pad2): track 0.00 -> 20.5 mm
- net Net-(R9-Pad2): track 0.00 -> 19.4 mm
- net Net-(R11-Pad2): track 0.00 -> 19.1 mm
- net Net-(U1-Pad15): track 0.00 -> 17.4 mm, vias 0 -> 4
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Other:
- net class HT added: clearance 0.4, trace_width 0.25, via_dia 0.8, via_drill 0.4

Commit message: Finished the board
Parts:
- added G***: LOGO, knss_logo:knss_logo, B.Cu at (151.1, 70.0)
- R1, R10, R11, R2, R3, R4, R5, R7, R8, R9: value 50k -> 47k
- moved Q8 27.5 mm to (153.4, 100.8), turned to 270 degrees
- moved Q9 27.4 mm to (153.4, 96.0), turned to 270 degrees
- moved Q10 27.4 mm to (153.4, 91.2), turned to 270 degrees
- moved Q3 27.2 mm to (127.3, 87.1), turned to 90 degrees
- moved Q4 27.1 mm to (127.3, 92.2), turned to 90 degrees
- moved Q5 27.0 mm to (127.3, 97.0), turned to 90 degrees
- moved R10 23.7 mm to (130.0, 63.8), turned to 0 degrees
- moved R2 23.3 mm to (130.0, 61.5), turned to 0 degrees
- moved R4 23.1 mm to (130.0, 59.2), turned to 0 degrees
- moved Q6 21.9 mm to (127.3, 101.9), turned to 90 degrees
- moved Q1 21.2 mm to (150.2, 84.6), turned to 0 degrees
- moved U1 19.4 mm to (151.0, 56.5), turned to 180 degrees
- moved Q2 18.6 mm to (136.9, 81.0), turned to 90 degrees
- moved Q7 17.5 mm to (148.8, 102.6), turned to 270 degrees
- moved U2 13.8 mm to (150.0, 37.6)
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Routing:
- net Net-(Q7-Pad2): track 0.00 -> 84.7 mm, vias 0 -> 2
- net Net-(Q8-Pad2): track 0.00 -> 73.2 mm, vias 0 -> 6
- net Net-(Q10-Pad2): track 0.00 -> 66.8 mm, vias 0 -> 2
- net Net-(Q6-Pad2): track 0.00 -> 64.6 mm
- net Net-(Q9-Pad2): track 0.00 -> 50.4 mm
- net Net-(Q1-Pad2): track 0.00 -> 49.6 mm, vias 0 -> 2
- net Net-(Q5-Pad2): track 0.00 -> 47.4 mm
- net Net-(Q4-Pad2): track 0.00 -> 39.1 mm
- net Net-(Q3-Pad2): track 0.00 -> 38.1 mm, vias 0 -> 2
- net /CLK: track 50.1 -> 12.9 mm, vias 4 -> 0
- net /LATCH: track 54.2 -> 18.6 mm, vias 6 -> 0
- net /DATA_OUT: track 37.6 -> 3.57 mm, vias 2 -> 0
- net Net-(R4-Pad2): track 5.15 -> 34.5 mm, vias 0 -> 2
- net Net-(R2-Pad2): track 11.8 -> 38.4 mm, vias 0 -> 2
- net Net-(R10-Pad2): track 23.5 -> 49.5 mm
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- added copper zone on B.Cu, net GND
- added copper zone on F.Cu, net GND
Other:
- rule trace_min: 0.2 -> 0.15
- rule via_min_size: 0.4 -> 0.6

Commit message: Revision 2
Parts:
- removed the C1 at (151.0, 49.8)
- removed the J2 at (137.4, 64.5)
- removed NIX1: NixieTube, Valve:Z5730M
- removed Q10: MMBTA42, Package_TO_SOT_SMD:SOT-23
- removed the U1 at (151.0, 56.5)
- added C0: 100n, Capacitor_SMD:C_0805_2012Metric, B.Cu at (151.0, 49.8)
- added J0: DB9_Male_MountingHoles, Connector_Dsub:DSUB-9_Female_Horizontal_P2.77x2.84mm_EdgePinOffset7.70mm_Housed_MountingHolesOffset9.12mm, F.Cu at (137.4, 64.5)
- added NIX0: NixieTube, Valve:Z5730M, F.Cu at (139.9, 93.3)
- added Q0: Q_NPN_BEC, Package_TO_SOT_SMD:SOT-23, B.Cu at (151.5, 85.5)
- added U0: 74HC595, Package_SO:SOP-16_4.55x10.3mm_P1.27mm, B.Cu at (151.0, 56.5)
- Q1, Q2, Q3, Q4, Q5, Q6, Q7, Q8, Q9: value MMBTA42 -> Q_NPN_BEC
- moved G*** 22.6 mm to (129.3, 75.9)
- moved Q6 21.0 mm to (148.2, 102.0), turned to 180 degrees
- moved Q1 14.2 mm to (136.5, 81.1), turned to 270 degrees
- moved Q2 11.6 mm to (127.5, 87.8), turned to 0 degrees
- moved Q3 5.97 mm to (127.5, 93.1), turned to 0 degrees
- moved Q4 5.59 mm to (127.5, 97.8), turned to 0 degrees
- moved Q5 5.47 mm to (127.5, 102.5), turned to 0 degrees
- moved Q8 4.89 mm to (153.3, 95.9), turned to 180 degrees
- moved Q9 4.76 mm to (153.3, 91.2), turned to 180 degrees
- moved Q7 4.49 mm to (153.3, 102.0), turned to 180 degrees
- renumbered C2 to C1, C3 to C2, C4 to C3, J3 to J2, R1 to R0, R2 to R1, R6 to R10, R3 to R2, R4 to R3, R5 to R4, R7 to R5, R8 to R6, R9 to R7, R10 to R8, R11 to R9, U2 to U1
Connections:
- Q1 pad 1: Net-(NIX1-Pad1) -> Net-(Q1-Pad1)
- Q1 pad 2: Net-(Q1-Pad2) -> GND
- Q1 pad 3: GND -> Net-(NIX0-Pad2)
- Q2 pad 1: Net-(NIX1-Pad2) -> Net-(Q2-Pad1)
- Q2 pad 2: Net-(Q2-Pad2) -> GND
- Q2 pad 3: GND -> Net-(NIX0-Pad3)
- Q3 pad 1: Net-(NIX1-Pad3) -> Net-(Q3-Pad1)
- Q3 pad 2: Net-(Q3-Pad2) -> GND
- Q3 pad 3: GND -> Net-(NIX0-Pad4)
- Q4 pad 1: Net-(NIX1-Pad4) -> Net-(Q4-Pad1)
- Q4 pad 2: Net-(Q4-Pad2) -> GND
- Q4 pad 3: GND -> Net-(NIX0-Pad5)
- Q5 pad 1: Net-(NIX1-Pad5) -> Net-(Q5-Pad1)
- Q5 pad 2: Net-(Q5-Pad2) -> GND
- Q5 pad 3: GND -> Net-(NIX0-Pad6)
- Q6 pad 1: Net-(NIX1-Pad6) -> Net-(Q6-Pad1)
- Q6 pad 2: Net-(Q6-Pad2) -> GND
- Q6 pad 3: GND -> Net-(NIX0-Pad7)
- Q7 pad 1: Net-(NIX1-Pad7) -> Net-(Q7-Pad1)
- Q7 pad 2: Net-(Q7-Pad2) -> GND
- Q7 pad 3: GND -> Net-(NIX0-Pad8)
- Q8 pad 1: Net-(NIX1-Pad8) -> Net-(Q8-Pad1)
- Q8 pad 2: Net-(Q8-Pad2) -> GND
- Q8 pad 3: GND -> Net-(NIX0-Pad9)
- Q9 pad 1: Net-(NIX1-Pad9) -> Net-(Q9-Pad1)
- Q9 pad 2: Net-(Q9-Pad2) -> GND
- Q9 pad 3: GND -> Net-(NIX0-Pad10)
- R0 pad 1: Net-(Q1-Pad2) -> Net-(Q0-Pad1)
- R1 pad 1: Net-(Q2-Pad2) -> Net-(Q1-Pad1)
- R2 pad 1: Net-(Q3-Pad2) -> Net-(Q2-Pad1)
- R3 pad 1: Net-(Q4-Pad2) -> Net-(Q3-Pad1)
- R4 pad 1: Net-(Q5-Pad2) -> Net-(Q4-Pad1)
- R5 pad 1: Net-(Q6-Pad2) -> Net-(Q5-Pad1)
- R6 pad 1: Net-(Q7-Pad2) -> Net-(Q6-Pad1)
- R7 pad 1: Net-(Q8-Pad2) -> Net-(Q7-Pad1)
- R8 pad 1: Net-(Q9-Pad2) -> Net-(Q8-Pad1)
- R9 pad 1: Net-(Q10-Pad2) -> Net-(Q9-Pad1)
Routing:
- net Net-(Q6-Pad1): track 0.00 -> 90.5 mm, vias 0 -> 2
- net Net-(Q7-Pad2): track 84.7 -> 0.00 mm, vias 2 -> 0
- net Net-(Q7-Pad1): track 0.00 -> 76.8 mm, vias 0 -> 6
- net Net-(Q8-Pad2): track 73.2 -> 0.00 mm, vias 6 -> 0
- net Net-(Q10-Pad2): track 66.8 -> 0.00 mm, vias 2 -> 0
- net Net-(Q5-Pad1): track 0.00 -> 65.0 mm
- net Net-(Q6-Pad2): track 64.6 -> 0.00 mm
- net Net-(Q9-Pad1): track 0.00 -> 60.9 mm, vias 0 -> 4
- net Net-(Q0-Pad1): track 0.00 -> 54.3 mm, vias 0 -> 2
- net Net-(Q9-Pad2): track 50.4 -> 0.00 mm
- net Net-(Q1-Pad2): track 49.6 -> 0.00 mm, vias 2 -> 0
- net Net-(Q4-Pad1): track 0.00 -> 48.7 mm
- net Net-(Q5-Pad2): track 47.4 -> 0.00 mm
- net Net-(Q8-Pad1): track 0.00 -> 45.5 mm, vias 0 -> 2
- net Net-(Q3-Pad1): track 0.00 -> 40.1 mm
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Other:
- board text added: "2019-10-11"
- board text added: "F. Piórski"
- board text added: "Rev. 2"
